Commit message: feat: original twip

File: tasks/twip/assets/twip.urdf (robot description, URDF)
Before this commit: robot twip, 3 links, 2 joints
Links:
- link body: mass 2.24123 -> 1.245; geometry collision mesh filename=meshes/twip.stl; visual mesh filename=meshes/twip.stl
- link left_wheel: mass 0.190998 -> 0.042; geometry collision mesh filename=meshes/wheel.stl; visual mesh filename=meshes/wheel.stl
- link right_wheel: mass 0.190998 -> 0.042; geometry collision mesh filename=meshes/wheel.stl; visual mesh filename=meshes/wheel.stl
Joints:
- joint lwheel: origin xyz=0.0509238 -0.0784359 -0.0289244 rpy=-3.14159 1.5708 0 -> xyz=0.069 0.0 0.0 rpy=-3.14159 1.5708 0
- joint rwheel: origin xyz=-0.219373 -0.078494 -0.0289244 rpy=1.66533e-16 1.5708 0 -> xyz=-0.069 0.0 0.0 rpy=1.66533e-16 1.5708 0
